File: kicad/datum/datum.kicad_pcb (KiCad board)
At the start: 2 copper layers, 80 x 35 mm, 16 parts

Commit message: Generation of production data
Parts:
- removed H2, H3: MountingHole_Pad, MountingHole:MountingHole_3.2mm_M3_Pad_Via
- removed the REF** at (75.0, -5.00)
- removed the REF** at (5.00, -5.00)
- removed TP1: TestPoint, TestPoint:TestPoint_Pad_D4.0mm
- added REF**: OSHW-Logo_7.5x8mm_SilkScreen, Symbol:OSHW-Logo_7.5x8mm_SilkScreen, F.Cu at (165.4, 91.6)
- G***: moved to F.Cu
- moved G*** 166.5 mm to (150.0, 100.0)
- moved H1 166.5 mm to (135.0, 100.0)
- moved H4 166.5 mm to (165.0, 100.0)
- moved REF** 166.5 mm to (140.0, 110.0)
- moved REF** 166.5 mm to (140.0, 95.0)
- moved REF** 166.5 mm to (150.0, 100.0)
- moved REF** 166.5 mm to (160.0, 110.0)
- moved REF** 166.5 mm to (160.0, 95.0)
- moved REF** 166.3 mm to (135.0, 114.7)
- moved G*** 165.4 mm to (150.0, 101.0)
- moved G*** 130.6 mm to (134.5, 92.3), turned to 0 degrees
Routing:
- net GND: track 34.6 -> 64.8 mm
- net (no net): track 24.0 -> 0.00 mm
Other:
- board size 80 x 35 mm -> 40 x 30 mm
- board text added: "Edge Metallization"
- board text added: "PickPlacer Datum Board based on LumenPnP"
- board text removed: "Lot Number Here On Back Silkscreen"
- board text removed: "PCB-0004 REV00"
- board text removed: "Plated along this flat edge"

Commit message: Switched to 0.5mm fiducial
Parts:
- G***: footprint index:logo_mask -> Project:logo_mask
- G***: footprint index:goblin -> Project:goblin
- G***: footprint index:cal-dot-grid -> Project:cal-dot-grid
- H1, H4: footprint MountingHole:MountingHole_3.2mm_M3_Pad_Via -> Project:MountingHole_3.2mm_M3_Pad_Via
- REF** (x4): footprint Fiducial:Fiducial_1mm_Mask3mm -> Project:Fiducial_1mm_Mask3mm
- REF**: value Fiducial_1mm_Mask2mm -> Fiducial_05mm_Mask2mm; footprint Fiducial:Fiducial_1mm_Mask2mm -> Project:Fiducial_05mm_Mask2mm
- REF**: footprint index:30mm-ruler -> Project:30mm-ruler
- REF**: footprint Symbol:OSHW-Logo_7.5x8mm_SilkScreen -> Project:OSHW-Logo_7.5x8mm_SilkScreen
Changed lines of the file:
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@@
   (net 0 "")
   (net 1 "GND")
-  (footprint "Fiducial:Fiducial_1mm_Mask3mm" (layer "F.Cu")
+  (footprint "Project:Fiducial_1mm_Mask3mm" (layer "F.Cu")
     (at 140 110)
     (descr "Circular Fiducial, 1mm bare copper, 3mm soldermask opening (recommended)")
@@
       (solder_mask_margin 1) (clearance 1.1))
   )
-  (footprint "Fiducial:Fiducial_1mm_Mask3mm" (layer "F.Cu")
+  (footprint "Project:Fiducial_1mm_Mask3mm" (layer "F.Cu")
     (at 140 95)
     (descr "Circular Fiducial, 1mm bare copper, 3mm soldermask opening (recommended)")
@@
       (solder_mask_margin 1) (clearance 1.1))
   )
-  (footprint "index:logo_mask" (layer "F.Cu")
+  (footprint "Project:logo_mask" (layer "F.Cu")
     (at 150 100)
     (attr through_hole)
@@
       ) (layer "F.Mask") (width 0.01) (fill solid))
   )
-  (footprint "MountingHole:MountingHole_3.2mm_M3_Pad_Via" (layer "F.Cu")
+  (footprint "Project:MountingHole_3.2mm_M3_Pad_Via" (layer "F.Cu")
     (at 135 100)
     (descr "Mounting Hole 3.2mm, M3")
@@
       (net 1 "GND") (pinfunction "1") (pintype "input"))
   )
-  (footprint "MountingHole:MountingHole_3.2mm_M3_Pad_Via" (layer "F.Cu")
+  (footprint "Project:MountingHole_3.2mm_M3_Pad_Via" (layer "F.Cu")
     (at 165 100)
     (descr "Mounting Hole 3.2mm, M3")
@@
       (net 1 "GND") (pinfunction "1") (pintype "input"))
   )
-  (footprint "Fiducial:Fiducial_1mm_Mask2mm" (layer "F.Cu")
+  (footprint "Project:Fiducial_05mm_Mask2mm" (layer "F.Cu")
     (at 150 100)
-    (descr "Circular Fiducial, 1mm bare copper, 2mm soldermask opening (Level A)")
+    (descr "Circular Fiducial, 0.5mm bare copper, 2mm soldermask opening (Level A)")
     (tags "fiducial")
     (attr smd)
@@
       (effects (font (size 1 1) (thickness 0.15)))
     )
-    (fp_text value "Fiducial_1mm_Mask2mm" (at 0 2) (layer "F.Fab")
+    (fp_text value "Fiducial_05mm_Mask2mm" (at 0 2) (layer "F.Fab")
       (effects (font (size 1 1) (thickness 0.15)))
     )
@@
     (fp_circle (center 0 0) (end 1.25 0) (layer "F.CrtYd") (width 0.05) (fill none))
     (fp_circle (center 0 0) (end 1 0) (layer "F.Fab") (width 0.1) (fill none))
-    (pad "" smd circle (at 0 0) (size 1 1) (layers "F.Cu" "F.Mask")
-      (solder_mask_margin 0.5) (clearance 0.6))
+    (pad "" smd circle (at 0 0) (size 0.5 0.5) (layers "F.Cu" "F.Mask")
+      (solder_mask_margin 0.75) (clearance 0.85))
   )
-  (footprint "index:30mm-ruler" (layer "F.Cu")
+  (footprint "Project:30mm-ruler" (layer "F.Cu")
     (at 135.006 114.6975)
     (attr through_hole)
@@
     (fp_line (start 28.00024 -0.0005) (end 28.00024 -1.0005) (layer "F.Mask") (width 0.15))
   )
-  (footprint "Fiducial:Fiducial_1mm_Mask3mm" (layer "F.Cu")
+  (footprint "Project:Fiducial_1mm_Mask3mm" (layer "F.Cu")
     (at 160 110)
     (descr "Circular Fiducial, 1mm bare copper, 3mm soldermask opening (recommended)")
@@
       (solder_mask_margin 1) (clearance 1.1))
   )
-  (footprint "Fiducial:Fiducial_1mm_Mask3mm" (layer "F.Cu")
+  (footprint "Project:Fiducial_1mm_Mask3mm" (layer "F.Cu")
     (at 160 95)
     (descr "Circular Fiducial, 1mm bare copper, 3mm soldermask opening (recommended)")
@@
       (solder_mask_margin 1) (clearance 1.1))
   )
-  (footprint "Symbol:OSHW-Logo_7.5x8mm_SilkScreen" (layer "F.Cu")
+  (footprint "Project:OSHW-Logo_7.5x8mm_SilkScreen" (layer "F.Cu")
     (at 165.4 91.6)
     (descr "Open Source Hardware Logo")
@@
       ) (layer "F.SilkS") (width 0.01) (fill solid))
   )
-  (footprint "index:goblin" (layer "F.Cu")
+  (footprint "Project:goblin" (layer "F.Cu")
     (at 134.5 92.3)
     (attr through_hole)
@@
       ) (layer "F.Mask") (width 0.01) (fill solid))
   )
-  (footprint "index:cal-dot-grid" (layer "B.Cu")
+  (footprint "Project:cal-dot-grid" (layer "B.Cu")
     (at 150 101 -90)
     (attr through_hole)
