File: kicad/ring-light/ringLight.kicad_pcb (KiCad board)
At the start: 2 copper layers, 40 x 50.2 mm, 36 parts, among them J1 Connector Vertical, J2 Connector Horizontal, U1 74AHCT1G32

Commit message: Changed buffer to schmitt trigger type
Parts:
- removed C10: 100nF, Capacitor_SMD:C_0805_2012Metric
- J1: value Connector Vertical -> Connector Top
- J2: value Connector Horizontal -> Connector Bot
- R1: value 330R -> 100R
- U1: value 74AHCT1G32 -> 74LVC1G17GW
- moved R1 2.64 mm to (157.6, 85.0), turned to 90 degrees
- moved C9 2.41 mm to (155.3, 87.4), turned to 0 degrees
- moved U1 1.30 mm to (155.2, 85.0)
Routing:
- net GND: track 60.2 -> 0.00 mm, vias 14 -> 27
- net +5V: track 173.7 -> 169.8 mm, vias 3 -> 1
- net Data_In_3V3: track 12.8 -> 15.2 mm, vias 0 -> 1
- net Net-(U1-Pad2): track 3.64 -> 2.49 mm
- net Data_In_5V: track 2.95 -> 2.39 mm
Other:
- board text removed: "PCB-0002-04"
