File: kicad/ring-light/ringLight.kicad_sch (KiCad schematic)
At the start: 24 parts, among them J1 Connector Top, J2 Connector Bot, U1 74AHCT1G32

Commit message: Changed buffer to schmitt trigger type
Parts:
- removed C8: 100nF, Capacitor_SMD:C_0805_2012Metric, symbol Device:C
- removed U1: 74AHCT1G32, Package_TO_SOT_SMD:SOT-353_SC-70-5, symbol 74xGxx:74AHCT1G32
- added U1: 74LVC1G17GW, Package_TO_SOT_SMD:SOT-353_SC-70-5, symbol 74xGxx:74AHCT1G126
- D1, D2, D3, D4, D5, D6, D7, D8: JLCPCB C114586 -> (none); LCSC C114586 -> C2843785
- R1: value 330R -> 100R; JLCPCB C17630 -> (none); LCSC C17630 -> C17408; Part # 0805W8F3300T5E -> 0805W8F1000T5E
Connections:
- net +5V: now also U1.5 (VCC)
- net Data_In_5V: now also U1.4
- net GND: now also U1.1, U1.3 (GND)
- net at R1.1: now also U1.2
Other:
- moved on the sheet: C9, R1
