File: kicad/vacuum-sensor/vacuum-sensor.kicad_pcb (KiCad board)
At the start: 2 copper layers, 37 x 14 mm, 13 parts, among them J1 Conn_01x04, U1 XGZP6857A100KPGPN, U2 XGZP6857A100KPGPN, U3 MIC5233-5.0YM5-TR

Commit message: Added second optionalk connector
Parts:
- added J2: Conn_01x04, Connector_JST:JST_XH_S4B-XH-A_1x04_P2.50mm_Horizontal, F.Cu at (129.2, 91.5)
Changed lines of the file:
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@@
+    )
+  )
+  (footprint "Connector_JST:JST_XH_S4B-XH-A_1x04_P2.50mm_Horizontal" (layer "F.Cu")
+    (at 129.25 91.475)
+    (descr "JST XH series connector, S4B-XH-A (http://www.jst-mfg.com/product/pdf/eng/eXH.pdf), generated with kicad-footprint-generator")
+    (tags "connector JST XH horizontal")
+    (property "Sheetfile" "vacuum-sensor.kicad_sch")
+    (property "Sheetname" "")
+    (attr through_hole)
+    (fp_text reference "J2" (at 3.75 -3.5) (layer "F.SilkS") hide
+      (effects (font (size 1 1) (thickness 0.15)))
+    )
+    (fp_text value "Conn_01x04" (at 3.75 10.4) (layer "F.Fab")
+      (effects (font (size 1 1) (thickness 0.15)))
+    )
+    (fp_text user "${REFERENCE}" (at 3.75 3.45) (layer "F.Fab")
+      (effects (font (size 1 1) (thickness 0.15)))
+    )
+    (fp_line (start 10.06 -2.41) (end 8.64 -2.41) (layer "F.SilkS") (width 0.12))
+    (fp_line (start 2.25 3.2) (end 2.25 8.7) (layer "F.SilkS") (width 0.12))
+    (fp_line (start 0 -1.5) (end -0.3 -2.1) (layer "F.SilkS") (width 0.12))
+    (fp_line (start 3.75 9.31) (end -2.56 9.31) (layer "F.SilkS") (width 0.12))
+    (fp_line (start -1.14 -2.41) (end -1.14 2.09) (layer "F.SilkS") (width 0.12))
+    (fp_line (start 7.25 3.2) (end 7.25 8.7) (layer "F.SilkS") (width 0.12))
+    (fp_line (start -0.3 -2.1) (end 0.3 -2.1) (layer "F.SilkS") (width 0.12))
+    (fp_line (start -1.14 2.09) (end 3.75 2.09) (layer "F.SilkS") (width 0.12))
+    (fp_line (start 2.25 8.7) (end 2.75 8.7) (layer "F.SilkS") (width 0.12))
+    (fp_line (start 0.25 3.2) (end -0.25 3.2) (layer "F.SilkS") (width 0.12))
+    (fp_line (start 4.75 8.7) (end 5.25 8.7) (layer "F.SilkS") (width 0.12))
+    (fp_line (start 10.06 9.31) (end 10.06 -2.41) (layer "F.SilkS") (width 0.12))
+    (fp_line (start -0.25 8.7) (end 0.25 8.7) (layer "F.SilkS") (width 0.12))
+    (fp_line (start 5.25 3.2) (end 4.75 3.2) (layer "F.SilkS") (width 0.12))
+    (fp_line (start 8.64 2.09) (end 3.75 2.09) (layer "F.SilkS") (width 0.12))
+    (fp_line (start 5.25 8.7) (end 5.25 3.2) (layer "F.SilkS") (width 0.12))
+    (fp_line (start 2.75 8.7) (end 2.75 3.2) (layer "F.SilkS") (width 0.12))
+    (fp_line (start -0.25 3.2) (end -0.25 8.7) (layer "F.SilkS") (width 0.12))
+    (fp_line (start 0.25 8.7) (end 0.25 3.2) (layer "F.SilkS") (width 0.12))
+    (fp_line (start -2.56 9.31) (end -2.56 -2.41) (layer "F.SilkS") (width 0.12))
+    (fp_line (start 0.3 -2.1) (end 0 -1.5) (layer "F.SilkS") (width 0.12))
+    (fp_line (start 7.75 3.2) (end 7.25 3.2) (layer "F.SilkS") (width 0.12))
+    (fp_line (start 3.75 9.31) (end 10.06 9.31) (layer "F.SilkS") (width 0.12))
+    (fp_line (start 7.25 8.7) (end 7.75 8.7) (layer "F.SilkS") (width 0.12))
+    (fp_line (start 7.75 8.7) (end 7.75 3.2) (layer "F.SilkS") (width 0.12))
+    (fp_line (start 8.64 -2.41) (end 8.64 2.09) (layer "F.SilkS") (width 0.12))
+    (fp_line (start -2.56 -2.41) (end -1.14 -2.41) (layer "F.SilkS") (width 0.12))
+    (fp_line (start 2.75 3.2) (end 2.25 3.2) (layer "F.SilkS") (width 0.12))
+    (fp_line (start 4.75 3.2) (end 4.75 8.7) (layer "F.SilkS") (width 0.12))
+    (fp_line (start -2.95 9.7) (end 10.45 9.7) (layer "F.CrtYd") (width 0.05))
+    (fp_line (start -2.95 -2.8) (end -2.95 9.7) (layer "F.CrtYd") (width 0.05))
+    (fp_line (start 10.45 -2.8) (end -2.95 -2.8) (layer "F.CrtYd") (width 0.05))
+    (fp_line (start 10.45 9.7) (end 10.45 -2.8) (layer "F.CrtYd") (width 0.05))
+    (fp_line (start -1.25 2.2) (end 3.75 2.2) (layer "F.Fab") (width 0.1))
+    (fp_line (start 9.95 9.2) (end 9.95 -2.3) (layer "F.Fab") (width 0.1))
+    (fp_line (start -2.45 -2.3) (end -1.25 -2.3) (layer "F.Fab") (width 0.1))
+    (fp_line (start -1.25 -2.3) (end -1.25 2.2) (layer "F.Fab") (width 0.1))
+    (fp_line (start 9.95 -2.3) (end 8.75 -2.3) (layer "F.Fab") (width 0.1))
+    (fp_line (start 0 1.2) (end 0.625 2.2) (layer "F.Fab") (width 0.1))
+    (fp_line (start 8.75 -2.3) (end 8.75 2.2) (layer "F.Fab") (width 0.1))
+    (fp_line (start 3.75 9.2) (end 9.95 9.2) (layer "F.Fab") (width 0.1))
+    (fp_line (start -2.45 9.2) (end -2.45 -2.3) (layer "F.Fab") (width 0.1))
+    (fp_line (start 8.75 2.2) (end 3.75 2.2) (layer "F.Fab") (width 0.1))
+    (fp_line (start 3.75 9.2) (end -2.45 9.2) (layer "F.Fab") (width 0.1))
+    (fp_line (start -0.625 2.2) (end 0 1.2) (layer "F.Fab") (width 0.1))
+    (pad "1" thru_hole roundrect (at 0 0) (size 1.7 1.95) (drill 0.95) (layers *.Cu *.Mask) (roundrect_rratio 0.1470588235)
+      (net 3 "Net-(J1-Pad1)") (pinfunction "Pin_1") (pintype "passive"))
+    (pad "2" thru_hole oval (at 2.5 0) (size 1.7 1.95) (drill 0.95) (layers *.Cu *.Mask)
+      (net 6 "Net-(C5-Pad1)") (pinfunction "Pin_2") (pintype "passive"))
+    (pad "3" thru_hole oval (at 5 0) (size 1.7 1.95) (drill 0.95) (layers *.Cu *.Mask)
+      (net 7 "Net-(C6-Pad1)") (pinfunction "Pin_3") (pintype "passive"))
+    (pad "4" thru_hole oval (at 7.5 0) (size 1.7 1.95) (drill 0.95) (layers *.Cu *.Mask)
+      (net 1 "GND") (pinfunction "Pin_4") (pintype "passive"))
+    (model "${KICAD6_3DMODEL_DIR}/Connector_JST.3dshapes/JST_XH_S4B-XH-A_1x04_P2.50mm_Horizontal.wrl"
+      (offset (xyz 0 0 0))
+      (scale (xyz 1 1 1))
+      (rotate (xyz 0 0 0))
     )
   )

Commit message: Minor changes
Parts:
- removed J2: Conn_01x04, Connector_JST:JST_XH_S4B-XH-A_1x04_P2.50mm_Horizontal
Other:
- board size 37 x 14 mm -> 38 x 14 mm
Changed lines of the file:
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@@
-    )
-  )
-  (footprint "Connector_JST:JST_XH_S4B-XH-A_1x04_P2.50mm_Horizontal" (layer "F.Cu")
-    (at 129.25 91.475)
-    (descr "JST XH series connector, S4B-XH-A (http://www.jst-mfg.com/product/pdf/eng/eXH.pdf), generated with kicad-footprint-generator")
-    (tags "connector JST XH horizontal")
-    (property "Sheetfile" "vacuum-sensor.kicad_sch")
-    (property "Sheetname" "")
-    (attr through_hole)
-    (fp_text reference "J2" (at 3.75 -3.5) (layer "F.SilkS") hide
-      (effects (font (size 1 1) (thickness 0.15)))
-    )
-    (fp_text value "Conn_01x04" (at 3.75 10.4) (layer "F.Fab")
-      (effects (font (size 1 1) (thickness 0.15)))
-    )
-    (fp_text user "${REFERENCE}" (at 3.75 3.45) (layer "F.Fab")
-      (effects (font (size 1 1) (thickness 0.15)))
-    )
-    (fp_line (start 10.06 -2.41) (end 8.64 -2.41) (layer "F.SilkS") (width 0.12))
-    (fp_line (start 2.25 3.2) (end 2.25 8.7) (layer "F.SilkS") (width 0.12))
-    (fp_line (start 0 -1.5) (end -0.3 -2.1) (layer "F.SilkS") (width 0.12))
-    (fp_line (start 3.75 9.31) (end -2.56 9.31) (layer "F.SilkS") (width 0.12))
-    (fp_line (start -1.14 -2.41) (end -1.14 2.09) (layer "F.SilkS") (width 0.12))
-    (fp_line (start 7.25 3.2) (end 7.25 8.7) (layer "F.SilkS") (width 0.12))
-    (fp_line (start -0.3 -2.1) (end 0.3 -2.1) (layer "F.SilkS") (width 0.12))
-    (fp_line (start -1.14 2.09) (end 3.75 2.09) (layer "F.SilkS") (width 0.12))
-    (fp_line (start 2.25 8.7) (end 2.75 8.7) (layer "F.SilkS") (width 0.12))
-    (fp_line (start 0.25 3.2) (end -0.25 3.2) (layer "F.SilkS") (width 0.12))
-    (fp_line (start 4.75 8.7) (end 5.25 8.7) (layer "F.SilkS") (width 0.12))
-    (fp_line (start 10.06 9.31) (end 10.06 -2.41) (layer "F.SilkS") (width 0.12))
-    (fp_line (start -0.25 8.7) (end 0.25 8.7) (layer "F.SilkS") (width 0.12))
-    (fp_line (start 5.25 3.2) (end 4.75 3.2) (layer "F.SilkS") (width 0.12))
-    (fp_line (start 8.64 2.09) (end 3.75 2.09) (layer "F.SilkS") (width 0.12))
-    (fp_line (start 5.25 8.7) (end 5.25 3.2) (layer "F.SilkS") (width 0.12))
-    (fp_line (start 2.75 8.7) (end 2.75 3.2) (layer "F.SilkS") (width 0.12))
-    (fp_line (start -0.25 3.2) (end -0.25 8.7) (layer "F.SilkS") (width 0.12))
-    (fp_line (start 0.25 8.7) (end 0.25 3.2) (layer "F.SilkS") (width 0.12))
-    (fp_line (start -2.56 9.31) (end -2.56 -2.41) (layer "F.SilkS") (width 0.12))
-    (fp_line (start 0.3 -2.1) (end 0 -1.5) (layer "F.SilkS") (width 0.12))
-    (fp_line (start 7.75 3.2) (end 7.25 3.2) (layer "F.SilkS") (width 0.12))
-    (fp_line (start 3.75 9.31) (end 10.06 9.31) (layer "F.SilkS") (width 0.12))
-    (fp_line (start 7.25 8.7) (end 7.75 8.7) (layer "F.SilkS") (width 0.12))
-    (fp_line (start 7.75 8.7) (end 7.75 3.2) (layer "F.SilkS") (width 0.12))
-    (fp_line (start 8.64 -2.41) (end 8.64 2.09) (layer "F.SilkS") (width 0.12))
-    (fp_line (start -2.56 -2.41) (end -1.14 -2.41) (layer "F.SilkS") (width 0.12))
-    (fp_line (start 2.75 3.2) (end 2.25 3.2) (layer "F.SilkS") (width 0.12))
-    (fp_line (start 4.75 3.2) (end 4.75 8.7) (layer "F.SilkS") (width 0.12))
-    (fp_line (start -2.95 9.7) (end 10.45 9.7) (layer "F.CrtYd") (width 0.05))
-    (fp_line (start -2.95 -2.8) (end -2.95 9.7) (layer "F.CrtYd") (width 0.05))
-    (fp_line (start 10.45 -2.8) (end -2.95 -2.8) (layer "F.CrtYd") (width 0.05))
-    (fp_line (start 10.45 9.7) (end 10.45 -2.8) (layer "F.CrtYd") (width 0.05))
-    (fp_line (start -1.25 2.2) (end 3.75 2.2) (layer "F.Fab") (width 0.1))
-    (fp_line (start 9.95 9.2) (end 9.95 -2.3) (layer "F.Fab") (width 0.1))
-    (fp_line (start -2.45 -2.3) (end -1.25 -2.3) (layer "F.Fab") (width 0.1))
-    (fp_line (start -1.25 -2.3) (end -1.25 2.2) (layer "F.Fab") (width 0.1))
-    (fp_line (start 9.95 -2.3) (end 8.75 -2.3) (layer "F.Fab") (width 0.1))
-    (fp_line (start 0 1.2) (end 0.625 2.2) (layer "F.Fab") (width 0.1))
-    (fp_line (start 8.75 -2.3) (end 8.75 2.2) (layer "F.Fab") (width 0.1))
-    (fp_line (start 3.75 9.2) (end 9.95 9.2) (layer "F.Fab") (width 0.1))
-    (fp_line (start -2.45 9.2) (end -2.45 -2.3) (layer "F.Fab") (width 0.1))
-    (fp_line (start 8.75 2.2) (end 3.75 2.2) (layer "F.Fab") (width 0.1))
-    (fp_line (start 3.75 9.2) (end -2.45 9.2) (layer "F.Fab") (width 0.1))
-    (fp_line (start -0.625 2.2) (end 0 1.2) (layer "F.Fab") (width 0.1))
-    (pad "1" thru_hole roundrect (at 0 0) (size 1.7 1.95) (drill 0.95) (layers *.Cu *.Mask) (roundrect_rratio 0.1470588235)
-      (net 3 "Net-(J1-Pad1)") (pinfunction "Pin_1") (pintype "passive"))
-    (pad "2" thru_hole oval (at 2.5 0) (size 1.7 1.95) (drill 0.95) (layers *.Cu *.Mask)
-      (net 6 "Net-(C5-Pad1)") (pinfunction "Pin_2") (pintype "passive"))
-    (pad "3" thru_hole oval (at 5 0) (size 1.7 1.95) (drill 0.95) (layers *.Cu *.Mask)
-      (net 7 "Net-(C6-Pad1)") (pinfunction "Pin_3") (pintype "passive"))
-    (pad "4" thru_hole oval (at 7.5 0) (size 1.7 1.95) (drill 0.95) (layers *.Cu *.Mask)
-      (net 1 "GND") (pinfunction "Pin_4") (pintype "passive"))
-    (model "${KICAD6_3DMODEL_DIR}/Connector_JST.3dshapes/JST_XH_S4B-XH-A_1x04_P2.50mm_Horizontal.wrl"
-      (offset (xyz 0 0 0))
-      (scale (xyz 1 1 1))
-      (rotate (xyz 0 0 0))
     )
   )
@@
     )
   )
-  (gr_line (start 149.5 97) (end 151.5 95) (layer "Edge.Cuts") (width 0.1))
-  (gr_line (start 114.5 95) (end 114.5 85) (layer "Edge.Cuts") (width 0.1))
-  (gr_line (start 149.5 83) (end 151.5 85) (layer "Edge.Cuts") (width 0.1))
-  (gr_line (start 114.5 85) (end 116.5 83) (layer "Edge.Cuts") (width 0.1))
-  (gr_line (start 116.5 83) (end 149.5 83) (layer "Edge.Cuts") (width 0.1))
-  (gr_line (start 151.5 85) (end 151.5 95) (layer "Edge.Cuts") (width 0.1))
-  (gr_line (start 114.5 95) (end 116.5 97) (layer "Edge.Cuts") (width 0.1))
-  (gr_line (start 149.5 97) (end 116.5 97) (layer "Edge.Cuts") (width 0.1))
+  (gr_line (start 114 88.9) (end 114 85) (layer "Edge.Cuts") (width 0.1))
+  (gr_arc (start 114 88.9) (mid 115.1 90) (end 114 91.1) (layer "Edge.Cuts") (width 0.1))
+  (gr_line (start 152 85) (end 152 88.9) (layer "Edge.Cuts") (width 0.1))
+  (gr_line (start 150 97) (end 152 95) (layer "Edge.Cuts") (width 0.1))
+  (gr_line (start 114 91.1) (end 114 95) (layer "Edge.Cuts") (width 0.1))
+  (gr_line (start 150 83) (end 152 85) (layer "Edge.Cuts") (width 0.1))
+  (gr_line (start 152 91.1) (end 152 95) (layer "Edge.Cuts") (width 0.1))
+  (gr_line (start 114 85) (end 116 83) (layer "Edge.Cuts") (width 0.1))
+  (gr_line (start 116 83) (end 150 83) (layer "Edge.Cuts") (width 0.1))
+  (gr_arc (start 152 91.1) (mid 150.9 90) (end 152 88.9) (layer "Edge.Cuts") (width 0.1))
+  (gr_line (start 114 95) (end 116 97) (layer "Edge.Cuts") (width 0.1))
+  (gr_line (start 150 97) (end 116 97) (layer "Edge.Cuts") (width 0.1))
   (gr_text "Vacuum-Sensor\nRevA\nSimonK" (at 150.5 88.75) (layer "B.SilkS")
     (effects (font (size 1 1) (thickness 0.2)) (justify left mirror))
@@
     (polygon
       (pts
-        (xy 151.5 97)
-        (xy 114.5 97)
-        (xy 114.5 83)
-        (xy 151.5 83)
+        (xy 152 97)
+        (xy 114 97)
+        (xy 114 83)
+        (xy 152 83)
       )
     )
@@
     (polygon
       (pts
-        (xy 151.5 97)
-        (xy 114.5 97)
-        (xy 114.5 83)
-        (xy 151.5 83)
+        (xy 152 97)
+        (xy 114 97)
+        (xy 114 83)
+        (xy 152 83)
       )
     )
