File: kicad/duet-encdb/duet-encdb.kicad_sch (KiCad schematic)
At the start: 27 parts, among them J1 Conn_02x05_Odd_Even, J2 Conn_01x08, J3 Conn_01x08, U1 LM2775DSG, U2 LM2775DSG, U3 74LVC541A

Commit message: Bumped to RevB, added series resistors to 10 pin header to not short out SPI pins during initialization
Parts:
- removed C7: 1u/10V, Capacitor_SMD:C_0603_1608Metric, symbol Device:C
- added R13, R14, R15, R16, R17, R18: 100R, Resistor_SMD:R_0603_1608Metric, symbol Device:R
Connections:
- net ENC1_A: now also R13.1; no longer U3.17 (Y1)
- net ENC1_B: now also R14.1; no longer U3.16 (Y2)
- net ENC1_N: now also R15.1; no longer U3.15 (Y3)
- net ENC2_A: now also R16.1; no longer U3.14 (Y4)
- net ENC2_B: now also R17.1; no longer U3.13 (Y5)
- net ENC2_N: now also R18.1; no longer U3.12 (Y6)
- new net: R17.2, U3.13 (Y5)
- new net: R15.2, U3.15 (Y3)
- new net: R16.2, U3.14 (Y4)
- new net: R18.2, U3.12 (Y6)
- new net: R14.2, U3.16 (Y2)
- new net: R13.2, U3.17 (Y1)

Commit message: Changed pinout of header, because for the CCL decoder to work, we need to place A and B signals on CCLIN and EXTINT pins simultaneously
Connections:
- net ENC1_N: now also J1.10 (Pin_10); no longer J1.7 (Pin_7)
- net ENC2_A: now also J1.7 (Pin_7)
- net ENC2_B: now also J1.3 (Pin_3)
- net ENC2_N: now also J1.6 (Pin_6); no longer J1.3 (Pin_3)
- no-connect marks 1 -> 0
Other:
- note added: "N/C"
- note added: "SPI1_CS0/EXTINT10 (PB10)"
- note added: "SPI1_CS2/EXTINT7 (PA07)"
- note removed: "SPI1_CS0/CCLIN11 (PB10)"
- note removed: "SPI1_CS2/AC_AIN3 (PA07)"
Changed lines of the file:
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@@
   (junction (at 152.4 88.9) (diameter 0) (color 0 0 0 0)
   )
-  (no_connect (at 78.74 50.8))
   (wire (pts (xy 73.66 107.95) (xy 73.66 104.775))
     (stroke (width 0) (type default) (color 0 0 0 0))
@@
     (stroke (width 0) (type default) (color 0 0 0 0))
   )
+  (wire (pts (xy 66.04 55.88) (xy 82.55 55.88))
+    (stroke (width 0) (type default) (color 0 0 0 0))
+  )
   (wire (pts (xy 149.86 83.82) (xy 163.83 83.82))
     (stroke (width 0) (type default) (color 0 0 0 0))
@@
     (effects (font (size 1.27 1.27)) (justify left bottom))
   )
+  (text "N/C" (at 85.09 55.88 0)
+    (effects (font (size 1.27 1.27)) (justify left bottom))
+  )
   (text "+5V" (at 214.63 95.25 0)
     (effects (font (size 1.27 1.27)) (justify left bottom))
@@
     (effects (font (size 1.27 1.27)) (justify left bottom))
   )
-  (text "SPI1_CS2/AC_AIN3 (PA07)" (at 15.24 53.34 0)
+  (text "SPI1_CS2/EXTINT7 (PA07)" (at 15.24 53.34 0)
     (effects (font (size 1.27 1.27)) (justify left bottom))
   )
@@
     (effects (font (size 1.27 1.27)) (justify left bottom))
   )
-  (text "SPI1_CS0/CCLIN11 (PB10)" (at 15.24 48.26 0)
+  (text "SPI1_CS0/EXTINT10 (PB10)" (at 15.24 48.26 0)
     (effects (font (size 1.27 1.27)) (justify left bottom))
   )
@@
     (effects (font (size 1.27 1.27)) (justify left bottom))
   )
-  (label "ENC1_N" (at 41.91 53.34 0)
+  (label "ENC1_N" (at 73.66 55.88 0)
     (effects (font (size 1.27 1.27)) (justify left bottom))
   )
@@
     (effects (font (size 1.27 1.27)) (justify left bottom))
   )
+  (label "ENC2_B" (at 41.91 48.26 0)
+    (effects (font (size 1.27 1.27)) (justify left bottom))
+  )
   (label "ENC2_N" (at 90.17 86.36 0)
     (effects (font (size 1.27 1.27)) (justify left bottom))
   )
-  (label "ENC2_N" (at 41.91 48.26 0)
-    (effects (font (size 1.27 1.27)) (justify left bottom))
-  )
+  (label "ENC2_N" (at 73.66 50.8 0)
+    (effects (font (size 1.27 1.27)) (justify left bottom))
+  )
+  (label "ENC2_A" (at 41.91 53.34 0)
+    (effects (font (size 1.27 1.27)) (justify left bottom))
+  )
