File: kicad/duet-encdb/duet-encdb.kicad_pcb (KiCad board)
At the start: 2 copper layers, 26 x 27 mm, 27 parts, among them J1 Conn_02x05_Odd_Even, J2 Conn_01x08, J3 Conn_01x08, U1 LM2775DSG, U2 LM2775DSG, U3 74LVC541A

Commit message: Bumped to RevB, added series resistors to 10 pin header to not short out SPI pins during initialization
Parts:
- removed C7: 1u/10V, Capacitor_SMD:C_0603_1608Metric
- added R13: 100R, Resistor_SMD:R_0603_1608Metric, F.Cu at (103.8, 95.5)
- added R14: 100R, Resistor_SMD:R_0603_1608Metric, F.Cu at (102.4, 95.5)
- added R15: 100R, Resistor_SMD:R_0603_1608Metric, F.Cu at (101.0, 95.5)
- added R16: 100R, Resistor_SMD:R_0603_1608Metric, F.Cu at (99.6, 95.5)
- added R17: 100R, Resistor_SMD:R_0603_1608Metric, F.Cu at (98.2, 95.5)
- added R18: 100R, Resistor_SMD:R_0603_1608Metric, F.Cu at (96.8, 95.5)
- moved R3 7.08 mm to (106.0, 80.5), turned to 0 degrees
- moved R4 7.08 mm to (94.0, 80.5), turned to 180 degrees
- moved R2 4.14 mm to (106.0, 83.5), turned to 0 degrees
- moved R5 4.14 mm to (94.0, 83.5), turned to 180 degrees
- moved R1 2.57 mm to (106.0, 86.5), turned to 0 degrees
- moved R6 2.57 mm to (94.0, 86.5), turned to 180 degrees
- moved U3 2.00 mm to (100.0, 89.5)
- moved R11 1.50 mm to (106.0, 79.0), turned to 0 degrees
- moved R8 1.50 mm to (94.0, 79.0), turned to 180 degrees
- moved C1 0.50 mm to (105.0, 90.0)
- moved C2 0.50 mm to (106.0, 96.2)
- moved C3 0.50 mm to (107.0, 90.0)
- moved C4 0.50 mm to (95.0, 94.2)
- moved C5 0.50 mm to (94.0, 88.0)
- moved C6 0.50 mm to (93.0, 94.2)
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Connections:
- U3 pad 12: /ENC2_N -> Net-(U3-Pad12)
- U3 pad 13: /ENC2_B -> Net-(U3-Pad13)
- U3 pad 14: /ENC2_A -> Net-(U3-Pad14)
- U3 pad 15: /ENC1_N -> Net-(U3-Pad15)
- U3 pad 16: /ENC1_B -> Net-(U3-Pad16)
- U3 pad 17: /ENC1_A -> Net-(U3-Pad17)
Routing:
- net +3V3: track 28.1 -> 38.7 mm, vias 4 -> 7
- net GND: track 28.6 -> 35.2 mm, vias 23 -> 22
- net Net-(J3-Pad3): track 15.7 -> 9.44 mm
- net Net-(J2-Pad7): track 13.0 -> 6.79 mm
- net Net-(R3-Pad1): track 2.74 -> 8.66 mm
- net Net-(U3-Pad6): track 2.74 -> 8.66 mm
- net Net-(J2-Pad5): track 14.1 -> 8.94 mm
- net /ENC1_N: track 10.6 -> 5.62 mm
- net Net-(J3-Pad5): track 16.4 -> 11.6 mm
- net Net-(U3-Pad17): track 0.00 -> 4.49 mm
- net Net-(U3-Pad16): track 0.00 -> 3.93 mm
- net Net-(U3-Pad15): track 0.00 -> 3.15 mm
- net Net-(R2-Pad1): track 3.09 -> 6.11 mm
- net Net-(U3-Pad7): track 3.09 -> 6.08 mm
- net Net-(U3-Pad12): track 0.00 -> 2.70 mm
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Other:
- board size 26 x 27 mm -> 27 x 27 mm
- board text added: "RevB"
- board text removed: "RevA"
- board text removed: "SimonK"

Commit message: Changed pinout of header, because for the CCL decoder to work, we need to place A and B signals on CCLIN and EXTINT pins simultaneously
Connections:
- J1 pad 10: unconnected-(J1-Pad10) -> /ENC1_N
- J1 pad 3: /ENC2_N -> /ENC2_B
- J1 pad 6: unconnected-(J1-Pad6) -> /ENC2_N
- J1 pad 7: /ENC1_N -> /ENC2_A
Routing:
- net /ENC2_N: track 13.1 -> 8.58 mm, vias 0 -> 1
- net /ENC2_B: track 9.08 -> 12.0 mm
- net /ENC1_N: track 5.62 -> 7.78 mm

Commit message: Changed naming of ENC0/1 to ENC1/2
Other:
- board text added: "ENC0"
- board text removed: "ENC2"
Changed lines of the file:
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@@
     (effects (font (size 1 1) (thickness 0.15)))
   )
-  (gr_text "ENC1" (at 110.75 77) (layer "F.SilkS")
+  (gr_text "ENC0" (at 110.75 77) (layer "F.SilkS")
     (effects (font (size 1 1) (thickness 0.2)))
   )
@@
     (effects (font (size 0.8 0.8) (thickness 0.15)) (justify left))
   )
-  (gr_text "ENC2" (at 89.25 77) (layer "F.SilkS")
+  (gr_text "ENC1" (at 89.25 77) (layer "F.SilkS")
     (effects (font (size 1 1) (thickness 0.2)))
   )
