File: kicad/toolhead-board/toolhead-board.kicad_pcb (KiCad board)
At the start: 2 copper layers, 53.5 x 65 mm, 46 parts, among them J1 Conn_02x12_Top_Bottom, J10 CAM, J11 DB9_Male_MountingHoles, J12 Conn_01x08, J2 ZM, J3 LM, J4 RM, J5 RGB, J6 VL, J7 VR, J8 ZES, J9 USB_C_Receptacle_USB2.0, U1 XGZP6857A100KPGPN, U2 XGZP6857A100KPGPN, U3 MIC5233-5.0YM5-TR, U4 74LVC1G17GW, U5 LMZM23601

Commit message: Added RS422 receiver
Parts:
- removed H1, H4: MountingHole, Project:MountingHole_3.2mm_M3
- added C11: 100nF, Capacitor_SMD:C_0603_1608Metric, F.Cu at (80.0, 56.0)
- added R11: 10R, Resistor_SMD:R_0805_2012Metric, F.Cu at (84.0, 56.0)
- added R12: 10R, Resistor_SMD:R_0805_2012Metric, F.Cu at (82.0, 56.0)
- added U6: UA9637, Package_SO:SO-8_3.9x4.9mm_P1.27mm, F.Cu at (82.0, 50.5)
- moved H2 15.0 mm to (114.5, 77.0)
- moved H6 13.3 mm to (111.5, 90.0)
- moved C1 6.76 mm to (104.7, 70.0)
- moved R2 4.26 mm to (104.7, 82.0), turned to 180 degrees
- moved H3 3.61 mm to (111.5, 64.0)
- moved R8 2.85 mm to (106.0, 57.5), turned to 180 degrees
- moved C2 2.28 mm to (104.7, 84.0)
- moved R1 2.00 mm to (104.7, 72.0), turned to 180 degrees
- moved R10 1.89 mm to (104.7, 78.0), turned to 180 degrees
- moved R9 1.83 mm to (104.7, 76.0), turned to 180 degrees
- moved R7 1.77 mm to (97.0, 57.5), turned to 180 degrees
- moved C4 1.70 mm to (104.7, 74.0)
- moved J10 1.58 mm to (82.5, 87.0)
- moved J8 1.58 mm to (82.5, 61.0)
- moved C3 0.50 mm to (108.8, 72.0)
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Connections:
- J1 pad 12: /VR -> /ENC-B
- J1 pad 19: GNDA -> /VL
- J1 pad 20: /PSL -> GNDA
- J1 pad 21: /ENC-B -> /PSL
- J1 pad 24: /VL -> /ENC-A
- J1 pad 7: +24V -> /VR
- J1 pad 8: /PSR -> +24V
- J1 pad 9: /ENC-A -> /PSR
- J11 pad 0: unconnected-(J11-Pad0) -> GND
- J12 pad 1: unconnected-(J12-Pad1) -> /A+
- J12 pad 2: unconnected-(J12-Pad2) -> /A-
- J12 pad 3: unconnected-(J12-Pad3) -> GND
- J12 pad 4: unconnected-(J12-Pad4) -> +5VD
- J12 pad 5: unconnected-(J12-Pad5) -> /B-
- J12 pad 6: unconnected-(J12-Pad6) -> /B+
- J12 pad 7: unconnected-(J12-Pad7) -> /Z-
- J12 pad 8: unconnected-(J12-Pad8) -> /Z+
Routing:
- net +5VD: track 15.9 -> 89.7 mm, vias 0 -> 3
- net /A+: track 0.00 -> 41.8 mm, vias 0 -> 1
- net Net-(C1-Pad1): track 0.00 -> 38.2 mm
- net /B+: track 0.00 -> 34.8 mm, vias 0 -> 1
- net /VL: track 35.4 -> 70.1 mm
- net /A-: track 0.00 -> 33.5 mm, vias 0 -> 1
- net /B-: track 0.00 -> 30.8 mm, vias 0 -> 1
- net /VR: track 10.7 -> 35.6 mm
- net /ENC-A: track 53.5 -> 68.5 mm, vias 0 -> 2
- net GND: track 0.00 -> 14.8 mm, vias 0 -> 12
- net GNDA: track 0.00 -> 13.4 mm, vias 0 -> 15
- net Net-(R1-Pad1): track 0.00 -> 12.3 mm
- net /PSL: track 16.7 -> 28.8 mm
- net /ENC-B: track 52.0 -> 63.5 mm, vias 0 -> 2
- net Net-(R2-Pad1): track 0.00 -> 8.00 mm
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- added copper zone on F.Cu, net GND
- added copper zone on F.Cu, net Net-(C9-Pad1)
Other:
- board size 53.5 x 65 mm -> 47.5 x 65 mm

Commit message: Final touches and gerber data generation
Parts:
- added R15: 10R, Resistor_SMD:R_0603_1608Metric, F.Cu at (104.7, 72.7)
- added R16: 10R, Resistor_SMD:R_0603_1608Metric, F.Cu at (104.7, 81.3)
- added U7: TLV6001DCK, Package_TO_SOT_SMD:SOT-353_SC-70-5, F.Cu at (108.8, 70.0)
- added U8: TLV6001DCK, Package_TO_SOT_SMD:SOT-353_SC-70-5, F.Cu at (108.8, 84.0)
- C11, C8: value 100nF -> 100n
- FB1: value FerriteBead -> 100R; footprint Inductor_SMD:L_0603_1608Metric -> Resistor_SMD:R_0805_2012Metric
- R1, R11, R12, R2, R3, R6, R7, R8: footprint Resistor_SMD:R_0805_2012Metric -> Resistor_SMD:R_0603_1608Metric
- R13: value 102K -> 100K
- R14: value 25.5K -> 24K
- moved R10 5.00 mm to (104.7, 83.0), turned to 0 degrees
- moved R9 5.00 mm to (104.7, 71.0), turned to 0 degrees
- moved H3 3.16 mm to (114.5, 63.0)
- moved H6 3.16 mm to (114.5, 91.0)
- moved R1 2.40 mm to (104.7, 74.4)
- moved R2 2.40 mm to (104.7, 79.6)
- moved C4 2.20 mm to (104.7, 76.2)
- moved C5 2.10 mm to (104.7, 77.9)
- moved R7 1.70 mm to (95.3, 57.5)
- moved R8 1.30 mm to (107.3, 57.5)
- moved C1 0.70 mm to (104.7, 69.3)
- moved C2 0.70 mm to (104.7, 84.7)
- moved C3 0.70 mm to (108.8, 72.7)
- moved U4 0.60 mm to (95.1, 79.5)
- moved C6 0.40 mm to (108.8, 79.4)
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Connections:
- C11 pad 1: +5VD -> GND
- C11 pad 2: GND -> +5VD
- R10 pad 2: /PSR -> Net-(R10-Pad2)
- R9 pad 2: /PSL -> Net-(R15-Pad1)
- U1 pad 4: Net-(R1-Pad1) -> Net-(R15-Pad1)
- U2 pad 4: Net-(R2-Pad1) -> Net-(R10-Pad2)
Routing:
- net Net-(R15-Pad1): track 0.00 -> 14.6 mm
- net Net-(R10-Pad2): track 0.00 -> 11.7 mm
- net Net-(C1-Pad1): track 38.2 -> 46.6 mm
- net Net-(R1-Pad1): track 12.3 -> 7.24 mm
- net GNDA: track 13.4 -> 18.2 mm, vias 15 -> 17
- net +24V: track 91.6 -> 93.6 mm
- net /ENC-B: track 63.5 -> 61.9 mm
- net /LM-B+: track 43.2 -> 41.9 mm
- net /A+: track 41.8 -> 40.7 mm
- net /ENC-A: track 68.5 -> 69.6 mm
- net /B+: track 34.8 -> 35.8 mm
- net /RGBSIG: track 34.7 -> 33.9 mm
- net /PSL: track 28.8 -> 28.1 mm
- net /LM-A+: track 36.3 -> 35.6 mm
- net Net-(R2-Pad1): track 8.00 -> 7.36 mm
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
Commit message: Moved mounting holes
Parts:
- moved H2 0.50 mm to (114.0, 77.0)
- moved H3 0.50 mm to (114.0, 63.0)
- moved H6 0.50 mm to (114.0, 91.0)
- moved C3 0.10 mm to (108.7, 72.7)
- moved C6 0.10 mm to (108.7, 79.4)
- moved R3 0.10 mm to (108.7, 81.5)
- moved U3 0.10 mm to (108.7, 75.9)
- moved U7 0.10 mm to (108.7, 70.0)
- moved U8 0.10 mm to (108.7, 84.0)

Commit message: Removed C7 on RGB line
Connections:
- J1 pad 11: /ZESR -> /ZESL
- J1 pad 23: /ZESL -> /ZESR
- J8 pad 1: /ZESR -> /ZESL
- J8 pad 4: /ZESL -> /ZESR
Routing:
- net /ZESR: track 45.6 -> 35.2 mm
- net /ZESL: track 35.2 -> 45.6 mm
Changed lines of the file:
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@@
     (fp_line (start -1.95 2.8) (end 7.95 2.8) (layer "F.Fab") (width 0.1))
     (pad "1" thru_hole roundrect (at 0 0 270) (size 1.2 1.75) (drill 0.75) (layers *.Cu *.Mask) (roundrect_rratio 0.2083333333)
-      (net 17 "/ZESR") (pinfunction "Pin_1") (pintype "passive"))
+      (net 16 "/ZESL") (pinfunction "Pin_1") (pintype "passive"))
     (pad "2" thru_hole oval (at 2 0 270) (size 1.2 1.75) (drill 0.75) (layers *.Cu *.Mask)
       (net 36 "GND") (pinfunction "Pin_2") (pintype "passive"))
@@
       (net 36 "GND") (pinfunction "Pin_3") (pintype "passive"))
     (pad "4" thru_hole oval (at 6 0 270) (size 1.2 1.75) (drill 0.75) (layers *.Cu *.Mask)
-      (net 16 "/ZESL") (pinfunction "Pin_4") (pintype "passive"))
+      (net 17 "/ZESR") (pinfunction "Pin_4") (pintype "passive"))
     (model "${KICAD6_3DMODEL_DIR}/Connector_JST.3dshapes/JST_PH_B4B-PH-K_1x04_P2.00mm_Vertical.wrl"
       (offset (xyz 0 0 0))
@@
     (property "Sheetfile" "toolhead-board.kicad_sch")
     (property "Sheetname" "")
-    (attr exclude_from_pos_files exclude_from_bom)
+    (attr exclude_from_pos_files)
     (fp_text reference "H5" (at 0 -4.2) (layer "F.SilkS") hide
       (effects (font (size 1 1) (thickness 0.15)))
@@
     (property "Sheetfile" "toolhead-board.kicad_sch")
     (property "Sheetname" "")
-    (attr exclude_from_pos_files exclude_from_bom)
+    (attr exclude_from_pos_files)
     (fp_text reference "H3" (at 0 -4) (layer "F.SilkS") hide
       (effects (font (size 1 1) (thickness 0.15)))
@@
     (property "Sheetfile" "toolhead-board.kicad_sch")
     (property "Sheetname" "")
-    (attr smd)
+    (attr smd exclude_from_pos_files exclude_from_bom)
     (fp_text reference "C7" (at 0 -1.43) (layer "F.SilkS") hide
       (effects (font (size 1 1) (thickness 0.15)))
@@
     (property "Sheetfile" "toolhead-board.kicad_sch")
     (property "Sheetname" "")
-    (attr exclude_from_pos_files exclude_from_bom)
+    (attr exclude_from_pos_files)
     (fp_text reference "H6" (at 0 -4.2) (layer "F.SilkS") hide
       (effects (font (size 1 1) (thickness 0.15)))
@@
       (net 9 "/RGBSIG") (pinfunction "Pin_10") (pintype "passive"))
     (pad "11" thru_hole circle (at 30 0 180) (size 1.5 1.5) (drill 1.02) (layers *.Cu *.Mask)
-      (net 17 "/ZESR") (pinfunction "Pin_11") (pintype "passive"))
+      (net 16 "/ZESL") (pinfunction "Pin_11") (pintype "passive"))
     (pad "12" thru_hole circle (at 33 0 180) (size 1.5 1.5) (drill 1.02) (layers *.Cu *.Mask)
       (net 39 "/ENC-B") (pinfunction "Pin_12") (pintype "passive"))
@@
       (net 36 "GND") (pinfunction "Pin_22") (pintype "passive"))
     (pad "23" thru_hole circle (at 30 3 180) (size 1.5 1.5) (drill 1.02) (layers *.Cu *.Mask)
-      (net 16 "/ZESL") (pinfunction "Pin_23") (pintype "passive"))
+      (net 17 "/ZESR") (pinfunction "Pin_23") (pintype "passive"))
     (pad "24" thru_hole circle (at 33 3 180) (size 1.5 1.5) (drill 1.02) (layers *.Cu *.Mask)
       (net 38 "/ENC-A") (pinfunction "Pin_24") (pintype "passive"))
@@
     (property "Sheetfile" "toolhead-board.kicad_sch")
     (property "Sheetname" "")
-    (attr exclude_from_pos_files exclude_from_bom)
+    (attr exclude_from_pos_files)
     (fp_text reference "H2" (at 0 -4) (layer "F.SilkS") hide
       (effects (font (size 1 1) (thickness 0.15)))
@@
   (segment (start 108.5 96.4) (end 108.5 97.75) (width 0.8) (layer "B.Cu") (net 15))
   (segment (start 118.1 61.9) (end 119.75 60.25) (width 0.8) (layer "B.Cu") (net 15))
-  (segment (start 91.995 96.245) (end 88 92.25) (width 0.4) (layer "B.Cu") (net 16))
-  (segment (start 82.55 68.55) (end 82.55 67) (width 0.4) (layer "B.Cu") (net 16))
-  (segment (start 88 92.25) (end 88 74) (width 0.4) (layer "B.Cu") (net 16))
-  (segment (start 88 74) (end 82.55 68.55) (width 0.4) (layer "B.Cu") (net 16))
-  (segment (start 91.995 97.915) (end 91.995 97.495) (width 0.5) (layer "B.Cu") (net 16))
-  (segment (start 91.995 97.915) (end 91.995 96.245) (width 0.4) (layer "B.Cu") (net 16))
-  (segment (start 81.6 61) (end 82.55 61) (width 0.4) (layer "B.Cu") (net 17))
-  (segment (start 87.25 92.5) (end 87.25 74.5) (width 0.4) (layer "B.Cu") (net 17))
-  (segment (start 90.5 95.75) (end 87.25 92.5) (width 0.4) (layer "B.Cu") (net 17))
-  (segment (start 90.5 99.42) (end 90.5 95.75) (width 0.4) (layer "B.Cu") (net 17))
-  (segment (start 81.1 61.5) (end 81.6 61) (width 0.4) (layer "B.Cu") (net 17))
-  (segment (start 81.1 68.35) (end 81.1 61.5) (width 0.4) (layer "B.Cu") (net 17))
-  (segment (start 87.25 74.5) (end 81.1 68.35) (width 0.4) (layer "B.Cu") (net 17))
-  (segment (start 91.995 100.915) (end 90.5 99.42) (width 0.4) (layer "B.Cu") (net 17))
+  (segment (start 81.6 61) (end 82.55 61) (width 0.4) (layer "B.Cu") (net 16))
+  (segment (start 87.25 92.5) (end 87.25 74.5) (width 0.4) (layer "B.Cu") (net 16))
+  (segment (start 90.5 95.75) (end 87.25 92.5) (width 0.4) (layer "B.Cu") (net 16))
+  (segment (start 90.5 99.42) (end 90.5 95.75) (width 0.4) (layer "B.Cu") (net 16))
+  (segment (start 81.1 61.5) (end 81.6 61) (width 0.4) (layer "B.Cu") (net 16))
+  (segment (start 81.1 68.35) (end 81.1 61.5) (width 0.4) (layer "B.Cu") (net 16))
+  (segment (start 87.25 74.5) (end 81.1 68.35) (width 0.4) (layer "B.Cu") (net 16))
+  (segment (start 91.995 100.915) (end 90.5 99.42) (width 0.4) (layer "B.Cu") (net 16))
+  (segment (start 91.995 96.245) (end 88 92.25) (width 0.4) (layer "B.Cu") (net 17))
+  (segment (start 82.55 68.55) (end 82.55 67) (width 0.4) (layer "B.Cu") (net 17))
+  (segment (start 88 92.25) (end 88 74) (width 0.4) (layer "B.Cu") (net 17))
+  (segment (start 88 74) (end 82.55 68.55) (width 0.4) (layer "B.Cu") (net 17))
+  (segment (start 91.995 97.915) (end 91.995 97.495) (width 0.5) (layer "B.Cu") (net 17))
+  (segment (start 91.995 97.915) (end 91.995 96.245) (width 0.4) (layer "B.Cu") (net 17))
   (segment (start 102.9 76.5) (end 102.9 81.5) (width 0.4) (layer "F.Cu") (net 18))
   (segment (start 103.875 72.7) (end 103.875 76.15) (width 0.4) (layer "F.Cu") (net 18))
