File: kicad/toolhead-board/toolhead-board.kicad_sch (KiCad schematic)
At the start: 46 parts, among them J1 Conn_02x12_Top_Bottom, J10 CAM, J11 DB9_Male_MountingHoles, J12 Conn_01x08, J2 ZM, J3 LM, J4 RM, J5 RGB, J6 VL, J7 VR, J8 ZES, J9 USB_C_Receptacle_USB2.0, U1 XGZP6857A100KPGPN, U2 XGZP6857A100KPGPN, U3 MIC5233-5.0YM5-TR, U4 74LVC1G17GW, U5 LMZM23601

Commit message: Added RS422 receiver
Parts:
- removed H1, H4: MountingHole, Project:MountingHole_3.2mm_M3, symbol Mechanical:MountingHole
- added C11: 100nF, Capacitor_SMD:C_0603_1608Metric, symbol Device:C
- added R11, R12: 10R, Resistor_SMD:R_0805_2012Metric, symbol Device:R
- added U6: UA9637, Package_SO:SO-8_3.9x4.9mm_P1.27mm, symbol Interface_LineDriver:UA9637
Connections:
- net +24V: now also J1.8 (Pin_8); no longer J1.7 (Pin_7)
- net +5VD: now also J12.4 (Pin_4), C11.1, U6.1 (VCC), U6.1 (VCC)
- net A+: now also J12.1 (Pin_1), U6.6 (IN+)
- net A-: now also J12.2 (Pin_2), U6.5 (IN-)
- net B+: now also J12.6 (Pin_6), U6.8 (IN+)
- net B-: now also J12.5 (Pin_5), U6.7 (IN-)
- net ENC-A: now also J1.24 (Pin_24), R11.2; no longer J1.9 (Pin_9)
- net ENC-B: now also J1.12 (Pin_12), R12.2; no longer J1.21 (Pin_21)
- net GND: now also J11.0 (PAD), J12.3 (Pin_3), C11.2, U6.4 (GND), U6.4 (GND)
- net GNDA: now also J1.20 (Pin_20); no longer J1.19 (Pin_19)
- net PSL: now also J1.21 (Pin_21); no longer J1.20 (Pin_20)
- net PSR: now also J1.9 (Pin_9); no longer J1.8 (Pin_8)
- net VL: now also J1.19 (Pin_19); no longer J1.24 (Pin_24)
- net VR: now also J1.7 (Pin_7); no longer J1.12 (Pin_12)
- net Z+: now also J12.8 (Pin_8)
- net Z-: now also J12.7 (Pin_7)
- new net: R12.1, U6.2 (OUT)
- new net: R11.1, U6.3 (OUT)
Other:
- moved on the sheet: C1, C2, C3, C4, C5, C6, C7, C8, H2, H3, H5, H6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

Commit message: Final touches and gerber data generation
Parts:
- added R15, R16: 10R, Resistor_SMD:R_0603_1608Metric, symbol Device:R
- added U7, U8: TLV6001DCK, Package_TO_SOT_SMD:SOT-353_SC-70-5, symbol Amplifier_Operational:TLV6001DCK
- C10: LCSC (none) -> C12891
- C11, C8: value 100nF -> 100n; JLCPCB C49678 -> (none); LCSC C49678 -> C14663; Part # CC0805KRX7R9BB104 -> (none)
- C9: LCSC (none) -> C13585
- FB1: value FerriteBead -> 100R; footprint Inductor_SMD:L_0603_1608Metric -> Resistor_SMD:R_0805_2012Metric; LCSC (none) -> C1015
- R1, R11, R12, R2, R3, R6, R7, R8: footprint Resistor_SMD:R_0805_2012Metric -> Resistor_SMD:R_0603_1608Metric
- R10, R4, R5, R9: LCSC (none) -> C23186
- R13: value 102K -> 100K; LCSC (none) -> C25803
- R14: value 25.5K -> 24K; LCSC (none) -> C23352
- U5: LCSC (none) -> C2861484
- U6: LCSC (none) -> C1544610
Connections:
- net +5VD: now also C11.2; no longer C11.1
- net GND: now also C11.1; no longer C11.2
- net GNDA: now also U7.2 (V-), U8.2 (V-)
- net PSL: now also R15.2; no longer R9.2
- net PSR: now also R16.2; no longer R10.2
- net at C1.1, C2.1, C3.1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: now also U7.5 (V+), U8.5 (V+)
- net at U2.4 (OUT): now also R10.2, R16.1, U8.1 (+); no longer R2.1
- net at U1.4 (OUT): now also R9.2, R15.1, U7.1 (+); no longer R1.1
- new net: R2.1, U8.3 (-), U8.4
- new net: R1.1, U7.3 (-), U7.4
Other:
- moved on the sheet: C2, C4, C5, R1, R10, R2, R9, U2

Commit message: Correct footprint for 0603 resistor
Parts:
- R1, R11, R12, R15, R16, R2, R3, R6, R7, R8: LCSC C17415 -> C22859
Changed lines of the file:
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@@
       (effects (font (size 1.27 1.27)) hide)
     )
-    (property "LCSC" "C17415" (id 4) (at 148.59 165.1 0)
+    (property "LCSC" "C22859" (id 4) (at 148.59 165.1 0)
       (effects (font (size 1.27 1.27)) hide)
     )
@@
       (effects (font (size 1.27 1.27)) hide)
     )
-    (property "LCSC" "C17415" (id 4) (at 107.95 62.23 0)
+    (property "LCSC" "C22859" (id 4) (at 107.95 62.23 0)
       (effects (font (size 1.27 1.27)) hide)
     )
@@
       (effects (font (size 1.27 1.27)) hide)
     )
-    (property "LCSC" "C17415" (id 4) (at 208.28 137.795 0)
+    (property "LCSC" "C22859" (id 4) (at 208.28 137.795 0)
       (effects (font (size 1.27 1.27)) hide)
     )
@@
       (effects (font (size 1.27 1.27)) hide)
     )
-    (property "LCSC" "C17415" (id 4) (at 107.315 97.79 0)
+    (property "LCSC" "C22859" (id 4) (at 107.315 97.79 0)
       (effects (font (size 1.27 1.27)) hide)
     )
@@
       (effects (font (size 1.27 1.27)) hide)
     )
-    (property "LCSC" "C17415" (id 4) (at 208.28 147.955 0)
+    (property "LCSC" "C22859" (id 4) (at 208.28 147.955 0)
       (effects (font (size 1.27 1.27)) hide)
     )
@@
       (effects (font (size 1.27 1.27)) hide)
     )
-    (property "LCSC" "C17415" (id 4) (at 107.95 71.755 0)
+    (property "LCSC" "C22859" (id 4) (at 107.95 71.755 0)
       (effects (font (size 1.27 1.27)) hide)
     )
@@
       (effects (font (size 1.27 1.27)) hide)
     )
-    (property "LCSC" "C17415" (id 4) (at 182.245 45.085 0)
+    (property "LCSC" "C22859" (id 4) (at 182.245 45.085 0)
       (effects (font (size 1.27 1.27)) hide)
     )
@@
       (effects (font (size 1.27 1.27)) hide)
     )
-    (property "LCSC" "C17415" (id 4) (at 148.59 137.795 0)
+    (property "LCSC" "C22859" (id 4) (at 148.59 137.795 0)
       (effects (font (size 1.27 1.27)) hide)
     )
@@
       (effects (font (size 1.27 1.27)) hide)
     )
-    (property "LCSC" "C17415" (id 4) (at 113.03 32.385 0)
+    (property "LCSC" "C22859" (id 4) (at 113.03 32.385 0)
       (effects (font (size 1.27 1.27)) hide)
     )
@@
       (effects (font (size 1.27 1.27)) hide)
     )
-    (property "LCSC" "C17415" (id 4) (at 107.315 107.95 0)
-      (effects (font (size 1.27 1.27)) hide)
-    )
+    (property "LCSC" "C22859" (id 4) (at 107.315 107.95 0)
+      (effects (font (size 1.27 1.27)) hide)
+    )

Commit message: Removed C7 on RGB line
Connections:
- net ZESL: now also J1.11 (Pin_11), J8.1 (Pin_1); no longer J1.23 (Pin_23), J8.4 (Pin_4)
- net ZESR: now also J1.23 (Pin_23), J8.4 (Pin_4); no longer J1.11 (Pin_11), J8.1 (Pin_1)
Other:
- moved on the sheet: J1
